File: PCB/Buzzard/Buzzard.kicad_pcb (KiCad board)
At the start: 0 parts

Commit message: started with pcb design and placed switches
Parts:
- added C1: 2.2uF, Buzzard:C_THT_SMD_0805_HandSolder_Reversable, F.Cu at (68.4, 259.2)
- added D1: D_Small, Buzzard:D3_TH_SMD_v2, F.Cu at (199.2, 121.8)
- added D10: D_Small, Buzzard:D3_TH_SMD_v2, F.Cu at (190.1, 124.1)
- added D11: D_Small, Buzzard:D3_TH_SMD_v2, F.Cu at (238.6, 85.5)
- added D12: D_Small, Buzzard:D3_TH_SMD_v2, F.Cu at (181.3, 124.1)
- added D13: D_Small, Buzzard:D3_TH_SMD_v2, F.Cu at (168.4, 121.8)
- added D14: D_Small, Buzzard:D3_TH_SMD_v2, F.Cu at (157.0, 133.6)
- added D15: D_Small, Buzzard:D3_TH_SMD_v2, F.Cu at (164.2, 135.9)
- added D16: D_Small, Buzzard:D3_TH_SMD_v2, F.Cu at (157.1, 131.3)
- added D17: D_Small, Buzzard:D3_TH_SMD_v2, F.Cu at (146.6, 136.2)
- added D18: D_Small, Buzzard:D3_TH_SMD_v2, F.Cu at (190.5, 121.8)
- added D19: D_Small, Buzzard:D3_TH_SMD_v2, F.Cu at (190.1, 131.0)
- added D2: D_Small, Buzzard:D3_TH_SMD_v2, F.Cu at (181.7, 121.8)
- added D20: D_Small, Buzzard:D3_TH_SMD_v2, F.Cu at (181.3, 131.0)
- added D3: D_Small, Buzzard:D3_TH_SMD_v2, F.Cu at (172.9, 135.1)
- added D4: D_Small, Buzzard:D3_TH_SMD_v2, F.Cu at (181.3, 128.7)
- added D5: D_Small, Buzzard:D3_TH_SMD_v2, F.Cu at (190.1, 128.7)
- added D6: D_Small, Buzzard:D3_TH_SMD_v2, F.Cu at (181.3, 126.4)
- added D7: D_Small, Buzzard:D3_TH_SMD_v2, F.Cu at (190.1, 126.4)
- added D8: D_Small, Buzzard:D3_TH_SMD_v2, F.Cu at (218.4, 103.6)
- added D9: D_Small, Buzzard:D3_TH_SMD_v2, F.Cu at (155.4, 136.2)
- added J1: PJ-320A, Buzzard:MJ-4PP-9, F.Cu at (-120.7, -5.68)
- added J2: SDA, Connector_PinHeader_2.54mm:PinHeader_1x01_P2.54mm_Vertical, F.Cu at (207.1, 170.8)
- added J3: SCL, Connector_PinHeader_2.54mm:PinHeader_1x01_P2.54mm_Vertical, F.Cu at (207.3, 176.9)
- added J4: Haptic Buzz, Connector_PinHeader_1.00mm:PinHeader_1x05_P1.00mm_Vertical, F.Cu at (69.7, 178.4)
- added J5: TrackPoint, Connector_PinHeader_1.00mm:PinHeader_1x05_P1.00mm_Vertical, F.Cu at (78.8, 259.8)
- added J6: OLED, Buzzard:OLED, F.Cu at (281.0, 145.8)
- added J7: LCD, Connector_PinHeader_1.00mm:PinHeader_1x08_P1.00mm_Vertical, F.Cu at (183.1, 317.1)
- added J8: Battery, Connector_JST:JST_PH_B2B-PH-K_1x02_P2.00mm_Vertical, F.Cu at (249.8, 174.7)
- added JP1: VCC Jumper, Jumper:SolderJumper-2_P1.3mm_Open_Pad1.0x1.5mm, F.Cu at (62.3, 175.8)
- added JP10: LCD CS Jumper, Jumper:SolderJumper-2_P1.3mm_Open_Pad1.0x1.5mm, F.Cu at (171.2, 324.9)
- added JP11: LCD CLK Jumper, Jumper:SolderJumper-2_P1.3mm_Open_Pad1.0x1.5mm, F.Cu at (194.7, 316.9)
- added JP12: LCD CS Jumper, Jumper:SolderJumper-2_P1.3mm_Open_Pad1.0x1.5mm, F.Cu at (195.0, 324.8)
- added JP13: GND Jumper, Jumper:SolderJumper-2_P1.3mm_Open_Pad1.0x1.5mm, F.Cu at (294.0, 129.9)
- added JP14: VCC Jumper, Jumper:SolderJumper-2_P1.3mm_Open_Pad1.0x1.5mm, F.Cu at (304.3, 129.5)
- added JP15: SCL Jumper, Jumper:SolderJumper-2_P1.3mm_Open_Pad1.0x1.5mm, F.Cu at (303.4, 137.8)
- added JP16: SDA Jumper, Jumper:SolderJumper-2_P1.3mm_Open_Pad1.0x1.5mm, F.Cu at (293.9, 137.7)
- added JP2: GND Jumper, Jumper:SolderJumper-2_P1.3mm_Open_Pad1.0x1.5mm, F.Cu at (61.6, 184.0)
- added JP3: VCC Jumper, Jumper:SolderJumper-2_P1.3mm_Open_Pad1.0x1.5mm, F.Cu at (78.1, 175.8)
- added JP4: GND Jumper, Jumper:SolderJumper-2_P1.3mm_Open_Pad1.0x1.5mm, F.Cu at (77.8, 184.7)
- added JP5: SDA Jumper, Jumper:SolderJumper-2_P1.3mm_Open_Pad1.0x1.5mm, F.Cu at (268.9, 134.5)
- added JP6: SCL Jumper, Jumper:SolderJumper-2_P1.3mm_Open_Pad1.0x1.5mm, F.Cu at (261.6, 134.3)
- added JP7: VCC Jumper, Jumper:SolderJumper-2_P1.3mm_Open_Pad1.0x1.5mm, F.Cu at (268.5, 128.3)
- added JP8: GND Jumper, Jumper:SolderJumper-2_P1.3mm_Open_Pad1.0x1.5mm, F.Cu at (259.0, 128.4)
- added JP9: LCD CLK Jumper, Jumper:SolderJumper-2_P1.3mm_Open_Pad1.0x1.5mm, F.Cu at (171.0, 317.3)
- added R1: 4.7kΩ, Buzzard:Resistor-TH_SMD, F.Cu at (77.6, 150.1)
- added R2: 4.7kΩ, Buzzard:Resistor-TH_SMD, F.Cu at (77.5, 146.9)
- added R3: 4.7kΩ, Buzzard:Resistor-TH_SMD, F.Cu at (57.5, 259.1)
- added R4: 4.7kΩ, Buzzard:Resistor-TH_SMD, F.Cu at (70.3, 265.3)
- added R5: 100kΩ, Buzzard:Resistor-TH_SMD, F.Cu at (57.2, 263.2)
- added S1: Switch, Buzzard:Kailh_socket_PG1350_optional_reversible.kicad_mod, F.Cu at (-91.9, -20.3)
- added S10: Switch, Buzzard:Kailh_socket_PG1350_optional_reversible.kicad_mod, F.Cu at (-51.7, -26.8)
- added S11: Switch, Buzzard:Kailh_socket_PG1350_optional_reversible.kicad_mod, F.Cu at (-45.9, -10.8)
- added S12: Switch, Buzzard:Kailh_socket_PG1350_optional_reversible.kicad_mod, F.Cu at (-67.4, 32.2)
- added S13: Switch, Buzzard:Kailh_socket_PG1350_optional_reversible.kicad_mod, F.Cu at (-34.1, -43.4)
- added S14: Switch, Buzzard:Kailh_socket_PG1350_optional_reversible.kicad_mod, F.Cu at (-29.7, -27.0)
- added S15: Switch, Buzzard:Kailh_socket_PG1350_optional_reversible.kicad_mod, F.Cu at (-25.3, -10.6)
- added S16: Switch, Buzzard:Kailh_socket_PG1350_optional_reversible.kicad_mod, F.Cu at (-5.93, -29.6)
- added S17: Switch, Buzzard:Kailh_socket_PG1350_optional_reversible.kicad_mod, F.Cu at (-4.45, -12.6)
- added S18: Switch, Buzzard:Kailh_socket_PG1350_optional_reversible.kicad_mod, F.Cu at (-2.97, 4.30)
- added S19: Switch, Buzzard:Kailh_socket_PG1350_optional_reversible.kicad_mod, F.Cu at (13.5, -14.2)
- added S2: Switch, Buzzard:Kailh_socket_PG1350_optional_reversible.kicad_mod, F.Cu at (-84.7, -4.94)
- added S20: Switch, Buzzard:Kailh_socket_PG1350_optional_reversible.kicad_mod, F.Cu at (15.0, 2.73)
- added S3: Switch, Buzzard:Kailh_socket_PG1350_optional_reversible.kicad_mod, F.Cu at (-77.6, 10.5)
- added S4: Switch, Buzzard:Kailh_socket_PG1350_optional_reversible.kicad_mod, F.Cu at (-96.9, 56.1)
- added S5: Switch, Buzzard:Kailh_socket_PG1350_optional_reversible.kicad_mod, F.Cu at (-76.5, -29.8)
- added S6: Switch, Buzzard:Kailh_socket_PG1350_optional_reversible.kicad_mod, F.Cu at (-69.2, -14.2)
- added S7: Switch, Buzzard:Kailh_socket_PG1350_optional_reversible.kicad_mod, F.Cu at (-62.1, 1.05)
- added S8: Switch, Buzzard:Kailh_socket_PG1350_optional_reversible.kicad_mod, F.Cu at (-83.7, 42.4)
- added S9: Switch, Buzzard:Kailh_socket_PG1350_optional_reversible.kicad_mod, F.Cu at (-57.5, -42.8)
- added SW1: SW_DPST_x2, Buzzard:SW-TH_3P-L9.1-W3.5-P2.50-S3.20-A3, F.Cu at (240.9, 175.2)
- added SW2: Reset, Buzzard:SMD-SW-4_5.1x5.1x2.5, F.Cu at (187.2, 174.3)
- added U1: ProMicro, Buzzard:ProMicro_v2, F.Cu at (-100.8, 5.14)
Other:
- board outline added: 150.4 x 122.8 mm
- copper layers 0 -> 2
